File: vr65816.kicad_pcb (KiCad board)
At the start: 2 copper layers, 150 x 125 mm, 79 parts, among them J1 PIX, J2 PWR&AMP, J3 GPIO, J4 AVOUT, J5 VGA, J6 AUDIO, SW1 REBOOT, U1 Pi Pico2W, U10 74AC04, U11 74HC4002, U12 74AC20, U13 74AC20, U2 Pi Pico2, U3 W65C816S, U4 W65C22S, U5 AS6C4008, U6 AS6C4008, U7 74AC245, U8 74AC573, U9 74AC00

Commit message: Add files via upload
Parts:
- removed R7: 47, vr65816:R_Axial_DIN0207_L6.3mm_D2.5mm_P10.16mm_Horizontal_Long
- R14: value 2k -> 220
- R5: value 2k -> 100
- moved C10 20.3 mm to (207.8, 106.5), turned to 90 degrees
- moved C9 20.3 mm to (207.8, 93.4), turned to 90 degrees
- moved C11 20.0 mm to (207.9, 109.6), turned to -90 degrees
- moved J3 16.9 mm to (70.0, 111.4)
- moved U10 12.6 mm to (204.1, 97.6), turned to -90 degrees
- moved U9 12.6 mm to (204.1, 84.4), turned to -90 degrees
- moved U11 12.4 mm to (204.2, 110.9), turned to -90 degrees
- moved J2 8.37 mm to (70.0, 75.9)
Connections:
- U10 pad 2: Net-(R7-Pad1) -> /PHI2B
- U10 pad 5: Net-(U10-Pad5) -> /A19
- U10 pad 6: /IRQB -> /AB17
- U9 pad 10: /A19 -> Net-(U9-Pad10)
- U9 pad 3: Net-(U10-Pad5) -> Net-(U9-Pad10)
- U9 pad 8: /AB17 -> /IRQB
- U9 pad 9: /A19 -> Net-(U9-Pad10)
Routing:
- net +3V3A: track 458.4 -> 400.3 mm, vias 3 -> 2
- net /AB17: track 82.7 -> 46.0 mm, vias 1 -> 0
- net /IRQB: track 128.8 -> 95.1 mm
- net Net-(U10-Pad5): track 32.0 -> 0.00 mm
- net /AB19: track 159.2 -> 128.8 mm
- net /A17: track 149.8 -> 121.2 mm
- net /A16: track 159.4 -> 133.8 mm
- net /IORQ: track 198.0 -> 221.4 mm
- net /PHI2B: track 58.7 -> 80.4 mm, vias 0 -> 2
- net /AB18: track 60.6 -> 39.3 mm
- net /A19: track 230.5 -> 211.8 mm, vias 3 -> 2
- net /RWB: track 292.8 -> 275.6 mm
- net Net-(R7-Pad1): track 17.0 -> 0.00 mm
- net Net-(U9-Pad10): track 0.00 -> 16.4 mm
- net /WEB: track 184.1 -> 199.6 mm
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