File: vr65816.kicad_pcb (KiCad board)
At the start: 2 copper layers, 150 x 125 mm, 78 parts, among them J1 PIX, J2 PWR&AMP, J3 GPIO, J4 AVOUT, J5 VGA, J6 AUDIO, SW1 REBOOT, U1 Pi Pico2W, U10 74AC04, U11 74HC4002, U12 74AC20, U13 74AC20, U2 Pi Pico2, U3 W65C816S, U4 W65C22S, U5 AS6C4008, U6 AS6C4008, U7 74AC245, U8 74AC573, U9 74AC00

Commit message: Add files via upload
Connections:
- U10 pad 10: /AB19 -> /AB17
- U10 pad 6: /AB17 -> /AB19
- U12 pad 2: /AB19 -> /AB17
- U12 pad 5: /AB17 -> /AB19
Routing:
- net /AB17: track 46.0 -> 28.6 mm
- net /A16: track 133.8 -> 127.7 mm
- net /AB18: track 39.3 -> 44.6 mm
- net /AB19: track 128.8 -> 124.6 mm
- net GND: track 1041.8 -> 1045.6 mm
- net /AB16: track 30.5 -> 28.7 mm
- net /A17: track 121.2 -> 122.0 mm
- net /A18: track 135.0 -> 135.6 mm
