File: vr65816.kicad_sch (KiCad schematic)
At the start: 74 parts, among them J1 PIX, J2 PWR&AMP, J3 GPIO, J4 AVOUT, J5 VGA, J6 AUDIO, SW1 REBOOT, U1 Pi Pico2W, U10 74AC04, U11 74HC4002, U12 74AC20, U13 74AC20, U2 Pi Pico2, U3 W65C816S, U4 W65C22S, U5 AS6C4008, U6 AS6C4008, U7 74AC245, U8 74AC573, U9 74AC00

Commit message: Add files via upload
Parts:
- removed R7: 47, vr65816:R_Axial_DIN0207_L6.3mm_D2.5mm_P10.16mm_Horizontal_Long, symbol Device:R
- R14: value 2k -> 220
- R5: value 2k -> 100
Connections:
- net A19: now also U10.5; no longer U9.10, U9.9
- net AB17: now also U10.6; no longer U9.8
- net IRQB: now also U9.8; no longer U10.6
- net PHI2B: now also U10.2
- net at U9.3: now also U9.10, U9.9; no longer U10.5
Other:
- moved on the sheet: U10A
