File: vr65816.kicad_sch (KiCad schematic)
At the start: 73 parts, among them J1 PIX, J2 PWR&AMP, J3 GPIO, J4 AVOUT, J5 VGA, J6 AUDIO, SW1 REBOOT, U1 Pi Pico2W, U10 74AC04, U11 74HC4002, U12 74AC20, U13 74AC20, U2 Pi Pico2, U3 W65C816S, U4 W65C22S, U5 AS6C4008, U6 AS6C4008, U7 74AC245, U8 74AC573, U9 74AC00

Commit message: Add files via upload
Connections:
- net AB17: now also U10.10, U12.2; no longer U10.6, U12.5
- net AB19: now also U10.6, U12.5; no longer U10.10, U12.2
Changed lines of the file:
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@@
 		)
 	)
-	(label "AB19"
+	(label "AB17"
 		(at 113.03 215.9 0)
 		(effects
@@
 		)
 	)
-	(label "AB17"
+	(label "AB19"
 		(at 113.03 220.98 0)
 		(effects
